Commit message: [robots] Fixed tiago_steel and tiago_titanium.

File: robots/tiago_steel.urdf (robot description, URDF)
Before this commit: robot tiago, 88 links, 87 joints
Links:
- removed link hand_grasping_frame
- removed link hand_index_abd_link
- removed link hand_index_flex_1_link
- removed link hand_index_flex_2_link
- removed link hand_index_flex_3_link
- removed link hand_index_link
- removed link hand_index_virtual_1_link
- removed link hand_index_virtual_2_link
- removed link hand_index_virtual_3_link
- removed link hand_little_abd_link
- removed link hand_little_flex_1_link
- removed link hand_little_flex_2_link
- removed link hand_little_flex_3_link
- removed link hand_little_virtual_1_link
- removed link hand_little_virtual_2_link
- removed link hand_little_virtual_3_link
- removed link hand_middle_abd_link
- removed link hand_middle_flex_1_link
- removed link hand_middle_flex_2_link
- removed link hand_middle_flex_3_link
- removed link hand_middle_virtual_1_link
- removed link hand_middle_virtual_2_link
- removed link hand_middle_virtual_3_link
- removed link hand_mrl_link
- removed link hand_palm_link
- removed link hand_ring_abd_link
- removed link hand_ring_flex_1_link
- removed link hand_ring_flex_2_link
- removed link hand_ring_flex_3_link
- removed link hand_ring_virtual_1_link
- removed link hand_ring_virtual_2_link
- removed link hand_ring_virtual_3_link
- removed link hand_safety_box
- removed link hand_thumb_abd_link
- removed link hand_thumb_flex_1_link
- removed link hand_thumb_flex_2_link
- removed link hand_thumb_link
- removed link hand_thumb_virtual_1_link
- removed link hand_thumb_virtual_2_link
- removed link hand_tool_link
- added link gripper_grasping_frame, mass 0.0001
- added link gripper_left_finger_link, mass 0.06286; collision box size=0.022 0.03 0.07; visual mesh filename=package://pal_wsg_gripper_description/meshes/gripper_finger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 scale=1 1 1
- added link gripper_left_fingertip_link, mass 0.000001
- added link gripper_link, mass 0.63871; collision mesh filename=package://pal_wsg_gripper_description/meshes/gripper_link_c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 scale=1 1 1; visual mesh filename=package://pal_wsg_gripper_description/meshes/gripper_link.s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 scale=1 1 1
- added link gripper_right_finger_link, mass 0.06286; collision box size=0.022 0.03 0.07; visual mesh filename=package://pal_wsg_gripper_description/meshes/gripper_finger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 scale=-1 -1 1
- added link gripper_right_fingertip_link, mass 0.000001
- added link gripper_tool_link, mass 0.0001
Joints:
- removed joint hand_grasping_fixed_joint
- removed joint hand_index_abd_joint
- removed joint hand_index_flex_1_joint
- removed joint hand_index_flex_2_joint
- removed joint hand_index_flex_3_joint
- removed joint hand_index_joint
- removed joint hand_index_virtual_1_joint
- removed joint hand_index_virtual_2_joint
- removed joint hand_index_virtual_3_joint
- removed joint hand_little_abd_joint
- removed joint hand_little_flex_1_joint
- removed joint hand_little_flex_2_joint
- removed joint hand_little_flex_3_joint
- removed joint hand_little_virtual_1_joint
- removed joint hand_little_virtual_2_joint
- removed joint hand_little_virtual_3_joint
- removed joint hand_middle_abd_joint
- removed joint hand_middle_flex_1_joint
- removed joint hand_middle_flex_2_joint
- removed joint hand_middle_flex_3_joint
- removed joint hand_middle_virtual_1_joint
- removed joint hand_middle_virtual_2_joint
- removed joint hand_middle_virtual_3_joint
- removed joint hand_mrl_joint
- removed joint hand_palm_joint
- removed joint hand_ring_abd_joint
- removed joint hand_ring_flex_1_joint
- removed joint hand_ring_flex_2_joint
- removed joint hand_ring_flex_3_joint
- removed joint hand_ring_virtual_1_joint
- removed joint hand_ring_virtual_2_joint
- removed joint hand_ring_virtual_3_joint
- removed joint hand_safety_box_joint
- removed joint hand_thumb_abd_joint
- removed joint hand_thumb_flex_1_joint
- removed joint hand_thumb_flex_2_joint
- removed joint hand_thumb_joint
- removed joint hand_thumb_virtual_1_joint
- removed joint hand_thumb_virtual_2_joint
- removed joint hand_tool_joint
- added joint gripper_finger_joint: type prismatic, parent gripper_link, child gripper_left_finger_link, origin xyz=-0.034 0.00000 0.00000 rpy=0.0 0.0 0.0, axis 1 0 0, limit lower=0.002 upper=0.034 effort=50 velocity=0.4
- added joint gripper_grasping_frame_joint: type fixed, parent gripper_link, child gripper_grasping_frame, origin xyz=0 0 -0.12 rpy=-1.5708 1.5708 0
- added joint gripper_joint: type fixed, parent wrist_ft_tool_link, child gripper_link, origin xyz=0.01 0 0 rpy=1.57079632679 1.57079632679 -1.57079632679, axis 0 0 0
- added joint gripper_left_fingertip_joint: type fixed, parent gripper_left_finger_link, child gripper_left_fingertip_link, origin xyz=0.035 0 -0.1465 rpy=0 -1.57079632679 0
- added joint gripper_right_finger_joint: type prismatic, parent gripper_link, child gripper_right_finger_link, origin xyz=0.034 0.00000 0.00000 rpy=0.0 0.0 0.0, axis -1 0 0, limit lower=0.002 upper=0.034 effort=16 velocity=0.4, mimic joint=gripper_finger_joint multiplier=1.0 offset=0.0
- added joint gripper_right_fingertip_joint: type fixed, parent gripper_right_finger_link, child gripper_right_fingertip_link, origin xyz=-0.035 0 -0.1465 rpy=0 1.57079632679 0
- added joint gripper_tool_joint: type fixed, parent wrist_ft_tool_link, child gripper_tool_link, origin xyz=0.01 0 0 rpy=1.57079632679 1.57079632679 -1.57079632679, axis 0 0 0

Commit message: [tiago_steel.urdf] Fix the joint type to be used in SoT.

File: robots/tiago_steel.urdf (robot description, URDF)
Before this commit: robot tiago, 55 links, 54 joints
Joints:
- joint caster_back_left_1_joint: type continuous -> fixed
- joint caster_back_left_2_joint: type continuous -> fixed
- joint caster_back_right_1_joint: type continuous -> fixed
- joint caster_back_right_2_joint: type continuous -> fixed
- joint caster_front_left_1_joint: type continuous -> fixed
- joint caster_front_left_2_joint: type continuous -> fixed
- joint caster_front_right_1_joint: type continuous -> fixed
- joint caster_front_right_2_joint: type continuous -> fixed
- joint suspension_left_joint: type prismatic -> fixed
- joint suspension_right_joint: type prismatic -> fixed
- joint wheel_left_joint: type continuous -> revolute
- joint wheel_right_joint: type continuous -> revolute

Commit message: [steel] Make some joints fixed.

File: robots/tiago_steel.urdf (robot description, URDF)
Before this commit: robot tiago, 55 links, 54 joints
Joints:
- joint caster_back_left_1_joint: type continuous -> fixed
- joint caster_back_left_2_joint: type continuous -> fixed
- joint caster_back_right_1_joint: type continuous -> fixed
- joint caster_back_right_2_joint: type continuous -> fixed
- joint caster_front_left_1_joint: type continuous -> fixed
- joint caster_front_left_2_joint: type continuous -> fixed
- joint caster_front_right_1_joint: type continuous -> fixed
- joint caster_front_right_2_joint: type continuous -> fixed
- joint gripper_right_finger_joint: type prismatic -> fixed
- joint suspension_left_joint: type prismatic -> fixed
- joint suspension_right_joint: type prismatic -> fixed
- joint wheel_left_joint: type continuous -> fixed
- joint wheel_right_joint: type continuous -> fixed

Commit message: Wheel joints are revolute.

File: robots/tiago_steel.urdf (robot description, URDF)
Before this commit: robot tiago, 55 links, 54 joints
Joints:
- joint wheel_left_joint: limit effort=6.0 velocity=10.152284264 -> lower=-inf upper=inf effort=6.0 velocity=10.152284264; type fixed -> revolute
- joint wheel_right_joint: limit effort=6.0 velocity=10.152284264 -> lower=-inf upper=inf effort=6.0 velocity=10.152284264; type fixed -> revolute

Commit message: [tiago_steel.urdf] Use same visual geometry for collision
  - head and arm collision geometries are not correct.

File: robots/tiago_steel.urdf (robot description, URDF)
Before this commit: robot tiago, 55 links, 54 joints
Links:
- link arm_1_link: geometry collision mesh filename=package://tiago_description/meshes/arm/arm_1.stl scale=1 1 1; visual mesh filename=package://tiago_description/meshes/arm/arm_1.stl scale=1 1 1
- link arm_2_link: geometry collision mesh filename=package://tiago_description/meshes/arm/arm_2.stl scale=1 1 1; visual mesh filename=package://tiago_description/meshes/arm/arm_2.stl scale=1 1 1
- link arm_3_link: geometry collision mesh filename=package://tiago_description/meshes/arm/arm_3.stl scale=1 1 1; visual mesh filename=package://tiago_description/meshes/arm/arm_3.stl scale=1 1 1
- link arm_4_link: geometry collision mesh filename=package://tiago_description/meshes/arm/arm_4.stl scale=1 1 1; visual mesh filename=package://tiago_description/meshes/arm/arm_4.stl scale=1 1 1
- link arm_5_link: geometry collision mesh filename=package://tiago_description/meshes/arm/arm_5.stl scale=1 1 1; visual mesh filename=package://tiago_description/meshes/arm/arm_5.stl scale=1 1 1
- link arm_6_link: geometry collision mesh filename=package://tiago_description/meshes/arm/arm_6.stl scale=1 1 1; visual mesh filename=package://tiago_description/meshes/arm/arm_6.stl scale=1 1 1
- link gripper_left_finger_link: geometry collision mesh filename=package://pal_wsg_gripper_description/meshes/gripper_finger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 scale=1 1 1; visual mesh filename=package://pal_wsg_gripper_description/meshes/gripper_finger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 scale=1 1 1
- link gripper_link: geometry collision mesh filename=package://pal_wsg_gripper_description/meshes/gripper_link.s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 scale=1 1 1; visual mesh filename=package://pal_wsg_gripper_description/meshes/gripper_link.s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 scale=1 1 1
- link gripper_right_finger_link: geometry collision mesh filename=package://pal_wsg_gripper_description/meshes/gripper_finger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 scale=-1 -1 1; visual mesh filename=package://pal_wsg_gripper_description/meshes/gripper_finger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 scale=-1 -1 1
- link head_1_link: geometry collision mesh filename=package://tiago_description/meshes/head/head_1.stl scale=1 1 1; visual mesh filename=package://tiago_description/meshes/head/head_1.stl scale=1 1 1
- link head_2_link: geometry collision mesh filename=package://tiago_description/meshes/head/head_2.stl scale=1 1 1; visual mesh filename=package://tiago_description/meshes/head/head_2.stl scale=1 1 1
- link torso_lift_link: geometry collision mesh filename=package://tiago_description/meshes/torso/torso_lift_with_ar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 scale=1 1 1; visual mesh filename=package://tiago_description/meshes/torso/torso_lift_with_ar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 scale=1 1 1

Commit message: Use Cylinder for base collision geometry.

File: robots/tiago_steel.urdf (robot description, URDF)
Before this commit: robot tiago, 55 links, 54 joints
Links:
- link base_link: geometry collision cylinder length=0.27 radius=.27; visual mesh filename=package://pmb2_description/meshes/base/base.stl

Commit message: Replace unsupported unbounded joint

File: robots/tiago_steel.urdf (robot description, URDF)
Before this commit: robot tiago, 55 links, 54 joints
Joints:
- joint wheel_left_joint: limit lower=-inf upper=inf effort=6.0 velocity=10.152284264 -> lower=-1.7976931348623157e+308 upper=1.7976931348623157e+308 effort=6.0 velocity=10.152284264
- joint wheel_right_joint: limit lower=-inf upper=inf effort=6.0 velocity=10.152284264 -> lower=-1.7976931348623157e+308 upper=1.7976931348623157e+308 effort=6.0 velocity=10.152284264

File: robots/tiago_steel_without_wheels.urdf (robot description, URDF)
Before this commit: robot tiago, 55 links, 54 joints
Joints:
- joint wheel_left_joint: limit lower=-inf upper=inf effort=6.0 velocity=10.152284264 -> effort=6.0 velocity=10.152284264
- joint wheel_right_joint: limit lower=-inf upper=inf effort=6.0 velocity=10.152284264 -> effort=6.0 velocity=10.152284264
